File: arduino-uno-connector/arduino-uno-connector.kicad_sch (KiCad schematic)
At the start: 10 parts, among them J2 Controller Connection, SW19 3V3 Switch, SW19 5V Switch, SW19 DIR_B / DIR_C, SW19 STP_B / STP_C

Commit message: Updated Printing for Arduino and GRBL Reference
Other:
- note added: "X"
- note added: "Y"
- note added: "Z"
Changed lines of the file:
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@@
     (effects (font (size 1.27 1.27)) (justify right bottom))
+  )
+  (text "Z" (at 81.28 81.28 0)
+    (effects (font (size 1.27 1.27)) (justify left bottom))
   )
   (text "spare" (at 87.63 160.02 0)
     (effects (font (size 1.27 1.27)) (justify right bottom))
   )
+  (text "Z" (at 81.28 88.9 0)
+    (effects (font (size 1.27 1.27)) (justify left bottom))
+  )
+  (text "Y\n" (at 81.28 78.74 0)
+    (effects (font (size 1.27 1.27)) (justify left bottom))
+  )
+  (text "X" (at 81.28 83.82 0)
+    (effects (font (size 1.27 1.27)) (justify left bottom))
+  )
+  (text "Y\n" (at 81.28 86.36 0)
+    (effects (font (size 1.27 1.27)) (justify left bottom))
+  )
+  (text "X" (at 81.28 76.2 0)
+    (effects (font (size 1.27 1.27)) (justify left bottom))
+  )
   (global_label "ENDSTOP_Z+" (shape input) (at 97.79 132.08 180) (fields_autoplaced)
     (effects (font (size 1.27 1.27)) (justify right))
@@
         )
       )
-      (project "arduino-connector"
+      (project "arduino-uno-connector"
         (path "/aa17e073-b1ff-4635-8f9d-ec77bbc3ea39"
           (reference "#PWR05") (unit 1)
@@
         )
       )
-      (project "arduino-connector"
+      (project "arduino-uno-connector"
         (path "/aa17e073-b1ff-4635-8f9d-ec77bbc3ea39"
           (reference "SW1") (unit 1)
@@
         )
       )
-      (project "arduino-connector"
+      (project "arduino-uno-connector"
         (path "/aa17e073-b1ff-4635-8f9d-ec77bbc3ea39"
           (reference "J1") (unit 1)
@@
     )
     (instances
-      (project "arduino-connector"
+      (project "arduino-uno-connector"
         (path "/aa17e073-b1ff-4635-8f9d-ec77bbc3ea39"
           (reference "H2") (unit 1)
@@
         )
       )
-      (project "arduino-connector"
+      (project "arduino-uno-connector"
         (path "/aa17e073-b1ff-4635-8f9d-ec77bbc3ea39"
           (reference "#PWR02") (unit 1)
@@
     )
     (instances
-      (project "arduino-connector"
+      (project "arduino-uno-connector"
         (path "/aa17e073-b1ff-4635-8f9d-ec77bbc3ea39"
           (reference "H1") (unit 1)
@@
         )
       )
-      (project "arduino-connector"
+      (project "arduino-uno-connector"
         (path "/aa17e073-b1ff-4635-8f9d-ec77bbc3ea39"
           (reference "#PWR06") (unit 1)
@@
         )
       )
-      (project "arduino-connector"
+      (project "arduino-uno-connector"
         (path "/aa17e073-b1ff-4635-8f9d-ec77bbc3ea39"
           (reference "SW3") (unit 1)
@@
         )
       )
-      (project "arduino-connector"
+      (project "arduino-uno-connector"
         (path "/aa17e073-b1ff-4635-8f9d-ec77bbc3ea39"
           (reference "#PWR03") (unit 1)
@@
     )
     (instances
-      (project "arduino-connector"
+      (project "arduino-uno-connector"
         (path "/aa17e073-b1ff-4635-8f9d-ec77bbc3ea39"
           (reference "H4") (unit 1)
@@
         )
       )
-      (project "arduino-connector"
+      (project "arduino-uno-connector"
         (path "/aa17e073-b1ff-4635-8f9d-ec77bbc3ea39"
           (reference "SW4") (unit 1)
@@
     (pin "1")
     (instances
-      (project "arduino-connector"
+      (project "arduino-uno-connector"
         (path "/aa17e073-b1ff-4635-8f9d-ec77bbc3ea39"
           (reference "#PWR01") (unit 1)
@@
     (pin "9")
     (instances
-      (project "arduino-connector"
+      (project "arduino-uno-connector"
         (path "/aa17e073-b1ff-4635-8f9d-ec77bbc3ea39"
           (reference "A1") (unit 1)
@@
         )
       )
-      (project "arduino-connector"
+      (project "arduino-uno-connector"
         (path "/aa17e073-b1ff-4635-8f9d-ec77bbc3ea39"
           (reference "#PWR04") (unit 1)
@@
         )
       )
-      (project "arduino-connector"
+      (project "arduino-uno-connector"
         (path "/aa17e073-b1ff-4635-8f9d-ec77bbc3ea39"
           (reference "SW2") (unit 1)
@@
     )
     (instances
-      (project "arduino-connector"
+      (project "arduino-uno-connector"
         (path "/aa17e073-b1ff-4635-8f9d-ec77bbc3ea39"
           (reference "H3") (unit 1)
